Commit message: Parameter adjustments for the vn100 IMU

File: config/robot.urdf.xacro (robot description, xacro)
@@ -21,4 +21,10 @@
     <origin xyz="0 0 0" rpy="0 0 0" />
   </joint>
+  <link name="velodyne"> </link>
+  <joint name="velodyne_joint" type="fixed">
+    <parent link="imu_link" />
+    <child link="velodyne" />
+    <origin xyz="0 0 0" rpy="0 0 0" />
+  </joint>
   <link name="laser_sensor_frame"> </link>
   <joint name="laser_joint" type="fixed">
